File: Lesson 4/EE-Workshop.sch (EAGLE design)
At the start: 1 part

Commit message: I made an piano
Parts:
- added IC1: NE555D, linear:NE555D
- added R1, R2, R3, R4, R5, R6: (no value), rcl:R-US_R0805
Changed lines of the file:
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@@
 <?xml version="1.0" encoding="utf-8"?>
 <!DOCTYPE eagle SYSTEM "eagle.dtd">
-<eagle version="9.2.2">
+<eagle version="9.4.0">
 <drawing>
 <settings>
@@
 <parts>
 <part name="BATT" library="battery" library_urn="urn:adsk.eagle:library:109" deviceset="AB9V" device="" package3d_urn="urn:adsk.eagle:package:4600/1" value="AB3V"/>
+<part name="IC1" library="linear" library_urn="urn:adsk.eagle:library:262" deviceset="*555" device="D" package3d_urn="urn:adsk.eagle:package:16404/2" technology="NE"/>
+<part name="R1" library="rcl" library_urn="urn:adsk.eagle:library:334" deviceset="R-US_" device="R0805" package3d_urn="urn:adsk.eagle:package:23553/2"/>
+<part name="R2" library="rcl" library_urn="urn:adsk.eagle:library:334" deviceset="R-US_" device="R0805" package3d_urn="urn:adsk.eagle:package:23553/2"/>
+<part name="R3" library="rcl" library_urn="urn:adsk.eagle:library:334" deviceset="R-US_" device="R0805" package3d_urn="urn:adsk.eagle:package:23553/2"/>
+<part name="R4" library="rcl" library_urn="urn:adsk.eagle:library:334" deviceset="R-US_" device="R0805" package3d_urn="urn:adsk.eagle:package:23553/2"/>
+<part name="R5" library="rcl" library_urn="urn:adsk.eagle:library:334" deviceset="R-US_" device="R0805" package3d_urn="urn:adsk.eagle:package:23553/2"/>
+<part name="R6" library="rcl" library_urn="urn:adsk.eagle:library:334" deviceset="R-US_" device="R0805" package3d_urn="urn:adsk.eagle:package:23553/2"/>
 </parts>
 <sheets>
@@
 <attribute name="NAME" x="19.685" y="47.625" size="1.778" layer="95" rot="R90"/>
 <attribute name="VALUE" x="27.94" y="47.625" size="1.778" layer="96" rot="R90"/>
+</instance>
+<instance part="IC1" gate="A" x="73.66" y="58.42" smashed="yes">
+<attribute name="NAME" x="66.04" y="69.342" size="1.778" layer="95"/>
+<attribute name="VALUE" x="66.04" y="45.593" size="1.778" layer="96"/>
+</instance>
+<instance part="R1" gate="G$1" x="40.64" y="20.32" smashed="yes">
+<attribute name="NAME" x="36.83" y="21.8186" size="1.778" layer="95"/>
+<attribute name="VALUE" x="36.83" y="17.018" size="1.778" layer="96"/>
+</instance>
+<instance part="R2" gate="G$1" x="27.94" y="20.32" smashed="yes">
+<attribute name="NAME" x="24.13" y="21.8186" size="1.778" layer="95"/>
+<attribute name="VALUE" x="24.13" y="17.018" size="1.778" layer="96"/>
+</instance>
+<instance part="R3" gate="G$1" x="15.24" y="20.32" smashed="yes">
+<attribute name="NAME" x="11.43" y="21.8186" size="1.778" layer="95"/>
+<attribute name="VALUE" x="11.43" y="17.018" size="1.778" layer="96"/>
+</instance>
+<instance part="R4" gate="G$1" x="53.34" y="20.32" smashed="yes">
+<attribute name="NAME" x="49.53" y="21.8186" size="1.778" layer="95"/>
+<attribute name="VALUE" x="49.53" y="17.018" size="1.778" layer="96"/>
+</instance>
+<instance part="R5" gate="G$1" x="68.58" y="20.32" smashed="yes">
+<attribute name="NAME" x="64.77" y="21.8186" size="1.778" layer="95"/>
+<attribute name="VALUE" x="64.77" y="17.018" size="1.778" layer="96"/>
+</instance>
+<instance part="R6" gate="G$1" x="83.82" y="20.32" smashed="yes">
+<attribute name="NAME" x="80.01" y="21.8186" size="1.778" layer="95"/>
+<attribute name="VALUE" x="80.01" y="17.018" size="1.778" layer="96"/>
 </instance>
 </instances>
@@
 packages will not be understood (or retained) with this version.
 </note>
+<note version="8.4" severity="warning">
+Since Version 8.4, EAGLE supports properties for SPICE simulation.
+Probes in schematics and SPICE mapping objects found in parts and library devices
+will not be understood with this version. Update EAGLE to the latest version
+for full support of SPICE simulation.
+</note>
 </compatibility>
